File: hardware/k30-SBC-dh/Bus.kicad_sch (KiCad schematic)
At the start: 31 parts, among them J4 ADBUS-EXP, J5 ADBUS, J6 SIGBUS, J7 POWER, J8 POWER, J9 POWER, U12 74HC393, U2 74HC14, U3 74HC05, U4 74HC139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

Commit message: use 5.08mm 1x2 screw terminal for power
These are good for 6A.

Noted on the silkscreen that this is a modified version
of the PCB.
Parts:
- removed J7, J8, J9: POWER, Connector_PinHeader_2.54mm:PinHeader_1x02_P2.54mm_Vertical, symbol Connector_Generic:Conn_01x02
- added J7: Screw_Terminal_01x02, TerminalBlock_CUI:TerminalBlock_CUI_TB007-508-02_1x02_P5.08mm_Horizontal, symbol Connector:Screw_Terminal_01x02
Connections:
- net +5V: now also J7.1 (Pin_1)
- net GND: now also J7.2 (Pin_2)
